Commit message: add missing xacro property deg_to_rad

File: urdf/d435.gazebo.xacro (robot description, xacro)
@@ -7,4 +7,5 @@
 <robot xmlns:xacro="http://ros.org/wiki/xacro">
   <xacro:macro name="simulation_d435" params="camera_name reference_link topics_ns depth_optical_frame color_optical_frame infrared1_optical_frame infrared2_optical_frame" >
+    <xacro:property name="deg_to_rad" value="0.017453292519943295"/>
     <!-- Load parameters to model's main link-->
     <gazebo reference="${reference_link}">
