Commit message: Update model files

File: urdf/d435.urdf (robot description, URDF)
Before this commit: robot d435, 10 links, 9 joints
Links:
- link camera_link: geometry collision box size=0.02505 0.09 0.025; visual mesh filename=package://d435/meshes/d435.dae

File: urdf/d435.urdf.xacro (robot description, xacro)
@@ -48,5 +48,5 @@
         <geometry>
           <!-- <box size="${d435_cam_width} ${d435_cam_height} ${d435_cam_depth}"/> -->
-	  <mesh filename="package://realsense2_camera/meshes/d435.dae" />
+	  <mesh filename="package://d435/meshes/d435.dae" />
           <!--<mesh filename="package://realsense2_camera/meshes/d435/d435.dae" />-->
         </geometry>
